Commit message: changes in urdf

File: catkin_ws/src/leap/description/robot.urdf (robot description, URDF)
Before this commit: robot onshape, 18 links, 16 joints
Links:
- removed link palm_lower
- added link base_link, mass 0.237; collision mesh filename=package://leap/description/palm_lower.stl; visual mesh filename=package://leap/description/palm_lower.stl
- link dip: geometry collision mesh filename=package://leap/description/dip.stl; visual mesh filename=package://leap/description/dip.stl
- link dip_2: geometry collision mesh filename=package://leap/description/dip.stl; visual mesh filename=package://leap/description/dip.stl
- link dip_3: geometry collision mesh filename=package://leap/description/dip.stl; visual mesh filename=package://leap/description/dip.stl
- link fingertip: geometry collision mesh filename=package://leap/description/fingertip.stl; visual mesh filename=package://leap/description/fingertip.stl
- link fingertip_2: geometry collision mesh filename=package://leap/description/fingertip.stl; visual mesh filename=package://leap/description/fingertip.stl
- link fingertip_3: geometry collision mesh filename=package://leap/description/fingertip.stl; visual mesh filename=package://leap/description/fingertip.stl
- link mcp_joint: geometry collision mesh filename=package://leap/description/mcp_joint.stl; visual mesh filename=package://leap/description/mcp_joint.stl
- link mcp_joint_2: geometry collision mesh filename=package://leap/description/mcp_joint.stl; visual mesh filename=package://leap/description/mcp_joint.stl
- link mcp_joint_3: geometry collision mesh filename=package://leap/description/mcp_joint.stl; visual mesh filename=package://leap/description/mcp_joint.stl
- link pip: geometry collision mesh filename=package://leap/description/pip.stl; visual mesh filename=package://leap/description/pip.stl
- link pip_2: geometry collision mesh filename=package://leap/description/pip.stl; visual mesh filename=package://leap/description/pip.stl
- link pip_3: geometry collision mesh filename=package://leap/description/pip.stl; visual mesh filename=package://leap/description/pip.stl
- link pip_4: geometry collision mesh filename=package://leap/description/pip.stl; visual mesh filename=package://leap/description/pip.stl
- link thumb_dip: geometry collision mesh filename=package://leap/description/thumb_dip.stl; visual mesh filename=package://leap/description/thumb_dip.stl
- link thumb_fingertip: geometry collision mesh filename=package://leap/description/thumb_fingertip.stl; visual mesh filename=package://leap/description/thumb_fingertip.stl
- link thumb_pip: geometry collision mesh filename=package://leap/description/thumb_pip.stl; visual mesh filename=package://leap/description/thumb_pip.stl
Joints:
- added joint virtual_joint: type fixed, parent world, child base_link, origin xyz=0 0 0.0 rpy=0 0 0
- joint 1: parent palm_lower -> base_link
- joint 12: parent palm_lower -> base_link
- joint 5: parent palm_lower -> base_link
- joint 9: parent palm_lower -> base_link

Commit message: moveit config error fixed

File: catkin_ws/src/leap/description/robot.urdf (robot description, URDF)
Before this commit: robot leap_hand, 18 links, 17 joints
Joints:
- removed joint 0
- removed joint 1
- removed joint 10
- removed joint 11
- removed joint 12
- removed joint 13
- removed joint 14
- removed joint 15
- removed joint 2
- removed joint 3
- removed joint 4
- removed joint 5
- removed joint 6
- removed joint 7
- removed joint 8
- removed joint 9
- added joint joint0: type revolute, parent mcp_joint, child pip, origin xyz=-0.012200000000000007713 0.038099999999999994982 0.014500000000000000736 rpy=-1.570796326794896558 -1.0065212660796336576e-15 1.5707963267948943376, axis 0 0 -1, limit lower=-1.047 upper=1.047 effort=0.95 velocity=8.48
- added joint joint1: type revolute, parent base_link, child mcp_joint, origin xyz=-0.0070952496528625457958 0.023057756134899472233 -0.01872240357846021927 rpy=1.5707963267948950037 1.5707963267948945596 0, axis 0 0 -1, limit lower=-0.314 upper=2.23 effort=0.95 velocity=8.48
- added joint joint10: type revolute, parent pip_3, child dip_3, origin xyz=0.014999999999999971689 0.014299999999999951639 -0.012999999999999959505 rpy=1.5707963267948958919 -1.570796326794896336 0, axis 0 0 -1, limit lower=-0.506 upper=1.885 effort=0.95 velocity=8.48
- added joint joint11: type revolute, parent dip_3, child fingertip_3, origin xyz=9.7144514654701197287e-17 -0.036099999999999868305 0.00020000000000007511769 rpy=4.5935029425113685044e-17 -2.8730071914463799514e-16 1.5565411607615035382e-32, axis 0 0 -1, limit lower=-0.366 upper=2.042 effort=0.95 velocity=8.48
- added joint joint12: type revolute, parent base_link, child pip_4, origin xyz=-0.069395249652862533996 -0.0012422438651005258004 -0.021622403578460215601 rpy=-8.2381766464939424156e-17 1.5707963267948956698 0, axis 0 0 -1, limit lower=-0.349 upper=2.094 effort=0.95 velocity=8.48
- added joint joint13: type revolute, parent pip_4, child thumb_pip, origin xyz=-2.7755575615628913511e-17 0.014300000000000005415 -0.013000000000000011546 rpy=1.5707963267948958919 -1.570796326794896336 0, axis 0 0 -1, limit lower=-0.47 upper=2.443 effort=0.95 velocity=8.48
- added joint joint14: type revolute, parent thumb_pip, child thumb_dip, origin xyz=0 0.014499999999999966041 -0.017000000000000053263 rpy=-1.570796326794896558 1.6050198443300131245e-46 -1.9721522630516624601e-31, axis 0 0 -1, limit lower=-1.20 upper=1.90 effort=0.95 velocity=8.48
- added joint joint15: type revolute, parent thumb_dip, child thumb_fingertip, origin xyz=-1.249000902703301108e-16 0.046599999999999863753 0.00019999999999997710581 rpy=1.5063958491491781023e-44 5.4234187233935260503e-31 3.141592653589793116, axis 0 0 -1, limit lower=-1.34 upper=1.88 effort=0.95 velocity=8.48
- added joint joint2: type revolute, parent pip, child dip, origin xyz=0.01499999999999996822 0.014299999999999904801 -0.012999999999999824196 rpy=1.5707963267948958919 -1.570796326794896336 0, axis 0 0 -1, limit lower=-0.506 upper=1.885 effort=0.95 velocity=8.48
- added joint joint3: type revolute, parent dip, child fingertip, origin xyz=-4.0880582495572692636e-09 -0.036100004210367367397 0.00020000000000007858714 rpy=4.5935029425113685044e-17 -2.8730071914463794583e-16 4.4395481053923607589e-32, axis 0 0 -1, limit lower=-0.366 upper=2.042 effort=0.95 velocity=8.48
- added joint joint4: type revolute, parent mcp_joint_2, child pip_2, origin xyz=-0.012200000000000019856 0.038099999999999981104 0.01450000000000000594 rpy=-1.570796326794896558 -1.0065212760057939085e-15 1.5707963267948943376, axis 0 0 -1, limit lower=-1.047 upper=1.047 effort=0.95 velocity=8.48
- added joint joint5: type revolute, parent base_link, child mcp_joint_2, origin xyz=-0.0070952496528625388569 -0.022392243865100525113 -0.018722403578460229678 rpy=1.570796326794896558 1.570796326794896558 0, axis 0 0 -1, limit lower=-0.314 upper=2.23 effort=0.95 velocity=8.48
- added joint joint6: type revolute, parent pip_2, child dip_2, origin xyz=0.014999999999999975159 0.014300000000000000211 -0.013000000000000018485 rpy=1.5707963267948958919 -1.570796326794896336 0, axis 0 0 -1, limit lower=-0.506 upper=1.885 effort=0.95 velocity=8.48
- added joint joint7: type revolute, parent dip_2, child fingertip_2, origin xyz=1.0061396160665481148e-16 -0.036099999999999854428 0.00020000000000007858714 rpy=4.5935029425113654229e-17 -2.8730071914463794583e-16 1.4408183216511868558e-31, axis 0 0 -1, limit lower=-0.366 upper=2.042 effort=0.95 velocity=8.48
- added joint joint8: type revolute, parent mcp_joint_3, child pip_3, origin xyz=-0.012200000000000004244 0.038100000000000001921 0.014499999999999999001 rpy=-1.570796326794896558 -1.0065212660796360242e-15 1.5707963267948943376, axis 0 0 -1, limit lower=-1.047 upper=1.047 effort=0.95 velocity=8.48
- added joint joint9: type revolute, parent base_link, child mcp_joint_3, origin xyz=-0.0070952454426398371343 -0.067842243865100515521 -0.018722407666402932774 rpy=1.5707963267948950037 1.5707963267948945596 0, axis 0 0 -1, limit lower=-0.314 upper=2.23 effort=0.95 velocity=8.48
